Commit message: Export the direct-drive robot hand, refresh the glove model, add glove-to-hand mapping
- Robot hand (Onshape element 354ca377…) exported to hand/ (URDF) and hand_mujoco/ (MJCF)
- Glove re-exported from the updated CAD (glove/, glove_mujoco/)
- glove_rules: weld grounded instances to the base (rule 4); treat a motor held by one
  cylinder + one non-coaxial parallel mate as fastened (rule 5)
- check_mates: orphaned bodies now count as a problem; per-joint body listing when they occur
- tune_mjcf / place_root / export_glove: use the exported robot's own directory instead of glove paths
- compare_kin: per-joint axis/sign/transmission comparison between glove and hand;
  writes config/glove_to_hand.json (sign + cubic phi(theta) per joint)
- find_rcm: virtual axis of the middle-finger double parallelogram
- twin_jog: two gloves in position mode with per-joint B offset trimming
- align_stops: align glove B zeros to glove A using mechanical stops
- calibrate: per-joint calibration by default (--whole-finger keeps the old flow)
- bilateral: per-joint follower gains, follower command low-pass, voltage display fix

Co-Authored-By: Claude Opus 5.5 <noreply@anthropic.com>

File: glove/robot.urdf (robot description, URDF)
Before this commit: robot glove, 66 links, 65 joints
Links:
- link part_1: mass 0.122037 -> 0.121822
